File: PCB/trippling_v1_2_moje.brd (EAGLE design)
At the start: 55.9 x 26.7 mm, 24 parts, among them K1 RELAY-SPDT-JZC-11F, K2 RELAY-SPDT-JZC-11F, T1 MMBT3904, T2 MMBT3904, X1 1751277

Commit message: Relay change
Parts:
- removed K1, K2: RELAY-SPDT-JZC-11F, SparkFun-Electromechanical:RELAY-JZC
- added K3, K4: 2071508-1, 2071508-1:RELAY_2071508-1
Connections:
- net +5V: now also K3.1, K4.1; no longer K1.5, K2.5
- net COM: now also K3.3, K4.3; no longer K1.3, K2.3
- net LEFT: now also K3.4; no longer K1.4
- net N$18: now also K3.2; no longer K1.1
- net N$21: now also K4.2; no longer K2.1
- net RIGHT: now also K4.4; no longer K2.4
Routing:
- net SET: track 10.4 -> 10.9 mm
