File: PCB/trippling_v1_2_moje.sch (EAGLE design)
At the start: 24 parts, among them K1 RELAY-SPDT-JZC-11F, K2 RELAY-SPDT-JZC-11F, T1 MMBT3904, T2 MMBT3904, X1 1751277

Commit message: Relay change
Parts:
- removed K1, K2: RELAY-SPDT-JZC-11F, SparkFun-Electromechanical:RELAY-SPDT-JZC-11F
- added K3, K4: 2071508-1, 2071508-1:2071508-1
Connections:
- net +5V: now also K3.COIL1, K4.COIL1; no longer K1.COIL1, K2.COIL1
- net COM: now also K3.NO, K4.NO; no longer K1.NO, K2.NO
- net LEFT: now also K3.COM; no longer K1.MAIN
- net N$18: now also K3.COIL2; no longer K1.COIL2
- net N$21: now also K4.COIL2; no longer K2.COIL2
- net RIGHT: now also K4.COM; no longer K2.MAIN
Changed lines of the file:
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@@
 <part name="D3" library="_hhn_diodes_smd" deviceset="1N4148WS" device="" override_package3d_urn="urn:adsk.eagle:package:24766019/2" override_package_urn="urn:adsk.eagle:footprint:24766020/1"/>
 <part name="RELE" library="SparkFun-DiscreteSemi" deviceset="ILD213T" device="-IDL213T" override_package3d_urn="urn:adsk.eagle:package:24766043/2" override_package_urn="urn:adsk.eagle:footprint:24766044/1"/>
-<part name="K1" library="SparkFun-Electromechanical" deviceset="RELAY-SPDT" device="-JZC-11F" override_package3d_urn="urn:adsk.eagle:package:24760025/2" override_package_urn="urn:adsk.eagle:footprint:24760066/1"/>
-<part name="K2" library="SparkFun-Electromechanical" deviceset="RELAY-SPDT" device="-JZC-11F" override_package3d_urn="urn:adsk.eagle:package:24761300/2" override_package_urn="urn:adsk.eagle:footprint:24761301/1"/>
 <part name="P+3" library="supply1" library_urn="urn:adsk.eagle:library:371" deviceset="+5V" device=""/>
 <part name="P+4" library="supply1" library_urn="urn:adsk.eagle:library:371" deviceset="+5V" device=""/>
@@
 <part name="P+9" library="supply1" library_urn="urn:adsk.eagle:library:371" deviceset="+5V" device=""/>
 <part name="C3" library="resistor" library_urn="urn:adsk.eagle:library:348" deviceset="C-EU" device="C0805" package3d_urn="urn:adsk.eagle:package:23617/2" value="100n"/>
+<part name="K3" library="2071508-1" deviceset="2071508-1" device="" override_package3d_urn="urn:adsk.eagle:package:24786443/2" override_package_urn="urn:adsk.eagle:footprint:24786444/1"/>
+<part name="K4" library="2071508-1" deviceset="2071508-1" device="" override_package3d_urn="urn:adsk.eagle:package:24786489/2" override_package_urn="urn:adsk.eagle:footprint:24786513/1"/>
 </parts>
 <sheets>
@@
 <attribute name="VALUE" x="17.78" y="17.272" size="1.778" layer="96" font="vector" align="top-left"/>
 </instance>
-<instance part="K1" gate="K$1" x="76.2" y="63.5" smashed="yes">
-<attribute name="NAME" x="68.58" y="71.374" size="1.778" layer="95" font="vector"/>
-<attribute name="VALUE" x="68.58" y="53.848" size="1.778" layer="96" font="vector"/>
-</instance>
-<instance part="K2" gate="K$1" x="76.2" y="12.7" smashed="yes">
-<attribute name="NAME" x="68.58" y="20.574" size="1.778" layer="95" font="vector"/>
-<attribute name="VALUE" x="68.58" y="3.048" size="1.778" layer="96" font="vector"/>
-</instance>
 <instance part="P+3" gate="1" x="66.04" y="78.74" smashed="yes">
 <attribute name="VALUE" x="63.5" y="73.66" size="1.778" layer="96" rot="R90"/>
@@
 <attribute name="NAME" x="-77.216" y="79.121" size="1.778" layer="95"/>
 <attribute name="VALUE" x="-77.216" y="74.041" size="1.778" layer="96"/>
+</instance>
+<instance part="K3" gate="G$1" x="78.74" y="63.5" smashed="yes">
+<attribute name="NAME" x="71.12" y="69.85" size="1.778" layer="95"/>
+<attribute name="VALUE" x="71.12" y="55.88" size="1.778" layer="96"/>
+</instance>
+<instance part="K4" gate="G$1" x="78.74" y="12.7" smashed="yes">
+<attribute name="NAME" x="71.12" y="19.05" size="1.778" layer="95"/>
+<attribute name="VALUE" x="71.12" y="5.08" size="1.778" layer="96"/>
 </instance>
 </instances>
@@
 <segment>
 <pinref part="P+3" gate="1" pin="+5V"/>
-<pinref part="K1" gate="K$1" pin="COIL1"/>
 <wire x1="66.04" y1="76.2" x2="66.04" y2="68.58" width="0.1524" layer="91"/>
 <pinref part="D3" gate="G$1" pin="C"/>
 <wire x1="66.04" y1="68.58" x2="58.42" y2="68.58" width="0.1524" layer="91"/>
 <wire x1="58.42" y1="68.58" x2="58.42" y2="66.04" width="0.1524" layer="91"/>
+<pinref part="K3" gate="G$1" pin="COIL1"/>
+<wire x1="66.04" y1="66.04" x2="66.04" y2="68.58" width="0.1524" layer="91"/>
 <junction x="66.04" y="68.58"/>
 </segment>
 <segment>
 <pinref part="P+4" gate="1" pin="+5V"/>
-<pinref part="K2" gate="K$1" pin="COIL1"/>
 <wire x1="66.04" y1="25.4" x2="66.04" y2="17.78" width="0.1524" layer="91"/>
 <pinref part="D2" gate="G$1" pin="C"/>
 <wire x1="66.04" y1="17.78" x2="58.42" y2="17.78" width="0.1524" layer="91"/>
 <wire x1="58.42" y1="17.78" x2="58.42" y2="15.24" width="0.1524" layer="91"/>
+<pinref part="K4" gate="G$1" pin="COIL1"/>
+<wire x1="66.04" y1="15.24" x2="66.04" y2="17.78" width="0.1524" layer="91"/>
 <junction x="66.04" y="17.78"/>
 </segment>
@@
 <net name="N$18" class="0">
 <segment>
-<pinref part="K1" gate="K$1" pin="COIL2"/>
 <pinref part="T2" gate="G$1" pin="C"/>
 <wire x1="66.04" y1="58.42" x2="66.04" y2="55.88" width="0.1524" layer="91"/>
@@
 <wire x1="66.04" y1="58.42" x2="58.42" y2="58.42" width="0.1524" layer="91"/>
 <wire x1="58.42" y1="58.42" x2="58.42" y2="60.96" width="0.1524" layer="91"/>
+<pinref part="K3" gate="G$1" pin="COIL2"/>
+<wire x1="66.04" y1="60.96" x2="66.04" y2="58.42" width="0.1524" layer="91"/>
 <junction x="66.04" y="58.42"/>
 </segment>
@@
 <segment>
 <pinref part="T1" gate="G$1" pin="C"/>
-<pinref part="K2" gate="K$1" pin="COIL2"/>
 <wire x1="66.04" y1="5.08" x2="66.04" y2="7.62" width="0.1524" layer="91"/>
 <pinref part="D2" gate="G$1" pin="A"/>
 <wire x1="66.04" y1="7.62" x2="58.42" y2="7.62" width="0.1524" layer="91"/>
 <wire x1="58.42" y1="7.62" x2="58.42" y2="10.16" width="0.1524" layer="91"/>
+<pinref part="K4" gate="G$1" pin="COIL2"/>
+<wire x1="66.04" y1="10.16" x2="66.04" y2="7.62" width="0.1524" layer="91"/>
 <junction x="66.04" y="7.62"/>
 </segment>
@@
 </segment>
 <segment>
-<pinref part="K1" gate="K$1" pin="MAIN"/>
-<wire x1="83.82" y1="63.5" x2="96.52" y2="63.5" width="0.1524" layer="91"/>
-<label x="86.36" y="63.5" size="1.778" layer="95"/>
+<wire x1="91.44" y1="66.04" x2="104.14" y2="66.04" width="0.1524" layer="91"/>
+<label x="93.98" y="66.04" size="1.778" layer="95"/>
+<pinref part="K3" gate="G$1" pin="COM"/>
 </segment>
 <segment>
@@
 <net name="RIGHT" class="0">
 <segment>
-<pinref part="K2" gate="K$1" pin="MAIN"/>
-<wire x1="96.52" y1="12.7" x2="83.82" y2="12.7" width="0.1524" layer="91"/>
-<label x="86.36" y="12.7" size="1.778" layer="95"/>
+<wire x1="104.14" y1="15.24" x2="91.44" y2="15.24" width="0.1524" layer="91"/>
+<label x="93.98" y="15.24" size="1.778" layer="95"/>
+<pinref part="K4" gate="G$1" pin="COM"/>
 </segment>
 <segment>
@@
 <net name="COM" class="0">
 <segment>
-<pinref part="K1" gate="K$1" pin="NO"/>
-<wire x1="83.82" y1="58.42" x2="96.52" y2="58.42" width="0.1524" layer="91"/>
-<label x="86.36" y="58.42" size="1.778" layer="95"/>
-</segment>
-<segment>
-<pinref part="K2" gate="K$1" pin="NO"/>
-<wire x1="83.82" y1="7.62" x2="96.52" y2="7.62" width="0.1524" layer="91"/>
-<label x="86.36" y="7.62" size="1.778" layer="95"/>
-</segment>
-<segment>
+<wire x1="91.44" y1="60.96" x2="104.14" y2="60.96" width="0.1524" layer="91"/>
+<label x="93.98" y="60.96" size="1.778" layer="95"/>
+<pinref part="K3" gate="G$1" pin="NO"/>
+</segment>
+<segment>
+<wire x1="91.44" y1="10.16" x2="104.14" y2="10.16" width="0.1524" layer="91"/>
+<label x="93.98" y="10.16" size="1.778" layer="95"/>
+<pinref part="K4" gate="G$1" pin="NO"/>
+</segment>
+<segment>
